File: KiCAD/Amiga-Card-Thru-Hole.kicad_pcb (KiCad board)
At the start: 2 copper layers, 170.2 x 107.1 mm, 20 parts, among them CN203 CN203, CN207 CN207, J1 Pi_0, J2 Push Button, U1 74AHC86N, U2 74LVC574A, U3 74LVC574A, U4 LD1117A, U5 SN74HC266N

Commit message: Add files via upload
Parts:
- removed R2: 1k, Resistor_THT:R_Axial_DIN0204_L3.6mm_D1.6mm_P7.62mm_Horizontal
- removed U5: SN74HC266N, Package_DIP:DIP-14_W7.62mm_Socket
- moved REF** 0.39 mm to (224.0, 87.0)
Connections:
- CN203 pad 12: GND -> Net-(CN203-Pad12)
- U1 pad 4: +3V3 -> /C1
- U1 pad 5: Net-(R2-Pad2) -> /C3
Routing:
- net Net-(R2-Pad2): track 70.6 -> 0.00 mm, vias 1 -> 0
- net /C1: track 33.9 -> 96.6 mm, vias 0 -> 2
- net +5V: track 292.4 -> 231.5 mm
- net GND: track 473.0 -> 420.6 mm
- net /C3: track 41.0 -> 61.2 mm, vias 0 -> 1
- net +3V3: track 180.4 -> 177.0 mm
Other:
- board text added: "Amiga Video Slot to Pi HDMI Rev. 1.1 Layout by jasonsbeer Original Amiga concept by c0pperdragon"
- board text removed: "Amiga Video Slot to Pi HDMI Rev. 1.0 Layout by jasonsbeer Original Amiga concept by c0pperdragon"
