File: KiCAD/Amiga-Card-Thru-Hole.sch (KiCad schematic (older format))
At the start: 17 parts, among them CN203 CN203, CN207 CN207, J1 Raspberry_Pi_0, J2 Push Button, U1 74AHC86N, U2 74LVC574A, U3 74LVC574A, U4 LD1117A, U5 SN74HC266N

Commit message: Add files via upload
Parts:
- removed R2: 1k, Resistor_THT:R_Axial_DIN0204_L3.6mm_D1.6mm_P7.62mm_Horizontal, symbol Device:R_Small
- removed U5: SN74HC266N, Package_DIP:DIP-14_W7.62mm_Socket, symbol 74xx_IEEE:74LS266
Connections:
- wire segments 132 -> 122
- no-connect marks 76 -> 74
Other:
- note added: "1.1"
- note added: "Amiga Video Slot to HDMI"
- moved on the sheet: U1E
Changed lines of the file:
@@
 	3250 5550 3250 5150
-Wire Wire Line
-	2650 5050 2650 4650
-$Comp
-L power:+3.3V #PWR0112
-U 1 1 60196E6C
-P 2650 4650
-F 0 "#PWR0112" H 2650 4500 50  0001 C CNN
-F 1 "+3.3V" H 2665 4823 50  0000 C CNN
-F 2 "" H 2650 4650 50  0001 C CNN
-F 3 "" H 2650 4650 50  0001 C CNN
-	1    2650 4650
-	1    0    0    -1
-$EndComp
 Wire Wire Line
 	3450 4050 4050 4050
@@
 $EndComp
 $Comp
-L power:GND #PWR0118
-U 1 1 602294B3
-P 2050 1350
-F 0 "#PWR0118" H 2050 1100 50  0001 C CNN
-F 1 "GND" H 2055 1177 50  0000 C CNN
-F 2 "" H 2050 1350 50  0001 C CNN
-F 3 "" H 2050 1350 50  0001 C CNN
-	1    2050 1350
-	0    -1   -1   0
-$EndComp
-$Comp
 L power:GND #PWR0120
 U 1 1 6022E2BA
@@
 L 74xx:74HC86 U1
 U 5 1 602A47FD
-P 6200 6850
-F 0 "U1" H 6200 7175 50  0000 C CNN
-F 1 "74AHC86N" H 6200 7084 50  0000 C CNN
-F 2 "Package_DIP:DIP-14_W7.62mm_Socket" H 6200 6850 50  0001 C CNN
-F 3 "http://www.ti.com/lit/gpn/sn74HC86" H 6200 6850 50  0001 C CNN
-	5    6200 6850
+P 1650 6450
+F 0 "U1" H 1650 6775 50  0000 C CNN
+F 1 "74AHC86N" H 1650 6684 50  0000 C CNN
+F 2 "Package_DIP:DIP-14_W7.62mm_Socket" H 1650 6450 50  0001 C CNN
+F 3 "http://www.ti.com/lit/gpn/sn74HC86" H 1650 6450 50  0001 C CNN
+	5    1650 6450
 	1    0    0    -1
 $EndComp
@@
 L power:GND #PWR0119
 U 1 1 602A723D
-P 6200 7350
-F 0 "#PWR0119" H 6200 7100 50  0001 C CNN
-F 1 "GND" H 6205 7177 50  0000 C CNN
-F 2 "" H 6200 7350 50  0001 C CNN
-F 3 "" H 6200 7350 50  0001 C CNN
-	1    6200 7350
+P 1650 6950
+F 0 "#PWR0119" H 1650 6700 50  0001 C CNN
+F 1 "GND" H 1655 6777 50  0000 C CNN
+F 2 "" H 1650 6950 50  0001 C CNN
+F 3 "" H 1650 6950 50  0001 C CNN
+	1    1650 6950
 	1    0    0    -1
 $EndComp
@@
 L power:+3.3V #PWR0121
 U 1 1 602A79AB
-P 6200 6350
-F 0 "#PWR0121" H 6200 6200 50  0001 C CNN
-F 1 "+3.3V" H 6215 6523 50  0000 C CNN
-F 2 "" H 6200 6350 50  0001 C CNN
-F 3 "" H 6200 6350 50  0001 C CNN
-	1    6200 6350
+P 1650 5950
+F 0 "#PWR0121" H 1650 5800 50  0001 C CNN
+F 1 "+3.3V" H 1665 6123 50  0000 C CNN
+F 2 "" H 1650 5950 50  0001 C CNN
+F 3 "" H 1650 5950 50  0001 C CNN
+	1    1650 5950
 	1    0    0    -1
 $EndComp
@@
 Text Label 2300 2450 0    50   ~ 0
 C1
-$Comp
-L power:GND #PWR0126
-U 1 1 602FA50C
-P 1700 6200
-F 0 "#PWR0126" H 1700 5950 50  0001 C CNN
-F 1 "GND" H 1705 6027 50  0000 C CNN
-F 2 "" H 1700 6200 50  0001 C CNN
-F 3 "" H 1700 6200 50  0001 C CNN
-	1    1700 6200
-	1    0    0    -1
-$EndComp
-$Comp
-L power:+5V #PWR0127
-U 1 1 602FB658
-P 2350 5350
-F 0 "#PWR0127" H 2350 5200 50  0001 C CNN
-F 1 "+5V" H 2365 5523 50  0000 C CNN
-F 2 "" H 2350 5350 50  0001 C CNN
-F 3 "" H 2350 5350 50  0001 C CNN
-	1    2350 5350
-	1    0    0    -1
-$EndComp
-Wire Wire Line
-	2650 5250 2650 5650
-Wire Wire Line
-	1200 6050 900  6050
-Wire Wire Line
-	1200 5850 900  5850
-$Comp
-L power:GND #PWR0128
-U 1 1 603152FE
-P 1500 7050
-F 0 "#PWR0128" H 1500 6800 50  0001 C CNN
-F 1 "GND" H 1505 6877 50  0000 C CNN
-F 2 "" H 1500 7050 50  0001 C CNN
-F 3 "" H 1500 7050 50  0001 C CNN
-	1    1500 7050
-	0    1    1    0
-$EndComp
-$Comp
-L power:GND #PWR0129
-U 1 1 60325CF3
-P 1500 7250
-F 0 "#PWR0129" H 1500 7000 50  0001 C CNN
-F 1 "GND" H 1505 7077 50  0000 C CNN
-F 2 "" H 1500 7250 50  0001 C CNN
-F 3 "" H 1500 7250 50  0001 C CNN
-	1    1500 7250
-	0    1    1    0
-$EndComp
-$Comp
-L power:GND #PWR0130
-U 1 1 6032649C
-P 4550 7050
-F 0 "#PWR0130" H 4550 6800 50  0001 C CNN
-F 1 "GND" H 4555 6877 50  0000 C CNN
-F 2 "" H 4550 7050 50  0001 C CNN
-F 3 "" H 4550 7050 50  0001 C CNN
-	1    4550 7050
-	0    1    1    0
-$EndComp
-$Comp
-L power:GND #PWR0131
-U 1 1 60326CD2
-P 4550 7250
-F 0 "#PWR0131" H 4550 7000 50  0001 C CNN
-F 1 "GND" H 4555 7077 50  0000 C CNN
-F 2 "" H 4550 7250 50  0001 C CNN
-F 3 "" H 4550 7250 50  0001 C CNN
-	1    4550 7250
-	0    1    1    0
-$EndComp
-$Comp
-L power:GND #PWR0132
-U 1 1 6032916A
-P 3100 7050
-F 0 "#PWR0132" H 3100 6800 50  0001 C CNN
-F 1 "GND" H 3105 6877 50  0000 C CNN
-F 2 "" H 3100 7050 50  0001 C CNN
-F 3 "" H 3100 7050 50  0001 C CNN
-	1    3100 7050
-	0    1    1    0
-$EndComp
-$Comp
-L power:GND #PWR0133
-U 1 1 6032993D
-P 3100 7250
-F 0 "#PWR0133" H 3100 7000 50  0001 C CNN
-F 1 "GND" H 3105 7077 50  0000 C CNN
-F 2 "" H 3100 7250 50  0001 C CNN
-F 3 "" H 3100 7250 50  0001 C CNN
-	1    3100 7250
-	0    1    1    0
-$EndComp
-Text Label 900  5850 0    50   ~ 0
+Wire Wire Line
+	2650 5250 2350 5250
+Wire Wire Line
+	2650 5050 2350 5050
+Text Label 2350 5050 0    50   ~ 0
 C1
-Text Label 900  6050 0    50   ~ 0
+Text Label 2350 5250 0    50   ~ 0
 C3
-$Comp
-L 74xx_IEEE:74LS266 U5
-U 1 1 603E3E2D
-P 1700 5950
-F 0 "U5" H 1700 6416 50  0000 C CNN
-F 1 "SN74HC266N" H 1700 6325 50  0000 C CNN
-F 2 "Package_DIP:DIP-14_W7.62mm_Socket" H 1700 5950 50  0001 C CNN
-F 3 "" H 1700 5950 50  0001 C CNN
-	1    1700 5950
-	1    0    0    -1
-$EndComp
-$Comp
-L 74xx_IEEE:74LS266 U5
-U 2 1 604329F5
-P 2000 7150
-F 0 "U5" H 2000 7616 50  0000 C CNN
-F 1 "SN74HC266N" H 2000 7525 50  0000 C CNN
-F 2 "Package_DIP:DIP-14_W7.62mm_Socket" H 2000 7150 50  0001 C CNN
-F 3 "" H 2000 7150 50  0001 C CNN
-	2    2000 7150
-	1    0    0    -1
-$EndComp
-$Comp
-L 74xx_IEEE:74LS266 U5
-U 3 1 6043AD24
-P 3600 7150
-F 0 "U5" H 3600 7616 50  0000 C CNN
-F 1 "SN74HC266N" H 3600 7525 50  0000 C CNN
-F 2 "Package_DIP:DIP-14_W7.62mm_Socket" H 3600 7150 50  0001 C CNN
-F 3 "" H 3600 7150 50  0001 C CNN
-	3    3600 7150
-	1    0    0    -1
-$EndComp
-NoConn ~ 2500 7150
-NoConn ~ 4100 7150
-$Comp
-L 74xx_IEEE:74LS266 U5
-U 4 1 6044A913
-P 5050 7150
-F 0 "U5" H 5050 7616 50  0000 C CNN
-F 1 "SN74HC266N" H 5050 7525 50  0000 C CNN
-F 2 "Package_DIP:DIP-14_W7.62mm_Socket" H 5050 7150 50  0001 C CNN
-F 3 "" H 5050 7150 50  0001 C CNN
-	4    5050 7150
-	1    0    0    -1
-$EndComp
-NoConn ~ 5550 7150
-$Comp
-L Device:R_Small R2
-U 1 1 603FD2B9
-P 2350 5450
-F 0 "R2" H 2409 5496 50  0000 L CNN
-F 1 "1k" H 2409 5405 50  0000 L CNN
-F 2 "Resistor_THT:R_Axial_DIN0204_L3.6mm_D1.6mm_P7.62mm_Horizontal" H 2350 5450 50  0001 C CNN
-F 3 "~" H 2350 5450 50  0001 C CNN
-	1    2350 5450
-	1    0    0    -1
-$EndComp
-Wire Wire Line
-	2350 5550 2350 5650
-Wire Wire Line
-	2350 5650 2650 5650
-Wire Wire Line
-	2200 5950 2350 5950
-Wire Wire Line
-	2350 5950 2350 5650
-Connection ~ 2350 5650
-Wire Wire Line
-	1700 5700 1700 5650
-Wire Wire Line
-	1700 5650 2150 5650
-Wire Wire Line
-	2150 5650 2150 5350
-Wire Wire Line
-	2150 5350 2350 5350
-Connection ~ 2350 5350
 $Comp
 L Connector:Conn_01x02_Male J2
@@
 Wire Wire Line
 	6750 4450 7600 4450
+NoConn ~ 2050 1350
+Text Notes 10600 7650 0    50   ~ 0
+1.1
+Text Notes 7350 7500 0    50   ~ 0
+Amiga Video Slot to HDMI
 $EndSCHEMATC
